File: arch/MGFieldHAT.kicad_pcb (KiCad board)
At the start: 2 copper layers, 65 x 30 mm, 10 parts

Commit message: added kicad file
Parts:
- removed the REF** at (155.5, 107.5)
- added DS18B20: TO-92-TO92127P495H2044-3, DS18B20 Footprint Symbol:TO-92-TO92127P495H2044-3, F.Cu at (153.5, 89.2)
- added DS18B20: TO-92-TO92127P495H2044-3, DS18B20 Footprint Symbol:TO-92-TO92127P495H2044-3, F.Cu at (142.7, 89.2)
- added FLC3-70: SolderWire-0.1sqmm_1x06_P3.6mm_D0.4mm_OD1mm, Connector_Wire:SolderWire-0.1sqmm_1x06_P3.6mm_D0.4mm_OD1mm, F.Cu at (138.0, 96.5)
- moved REF** 5.52 mm to (155.5, 79.0)
- moved REF** 5.52 mm to (149.5, 79.0)
- moved 4.7k 2.66 mm to (138.0, 80.1)
Routing:
- net (no net): track 0.00 -> 118.7 mm
- net GND: track 43.2 -> 75.5 mm
- net +5V: track 86.1 -> 113.3 mm
- net /GPIO4/GPCLK0: track 74.2 -> 55.2 mm
Other:
- board text added: "A0"
- board text added: "A1"
- board text added: "A2"
- board text added: "A3"
- board text added: "GND"
- board text added: "VCC"
